Commit message: update

File: scara_ws/src/scara_description/phold.urdf (robot description, URDF)
Before this commit: robot scara, 8 links, 7 joints
Links:
- link AL: geometry collision mesh filename=file://PLACEHOLDER/AL.STL; visual mesh filename=file://PLACEHOLDER/AL.STL
- link XL: geometry collision mesh filename=file://PLACEHOLDER/XL.STL; visual mesh filename=file://PLACEHOLDER/XL.STL
- link YL: geometry collision mesh filename=file://PLACEHOLDER/YL.STL; visual mesh filename=file://PLACEHOLDER/YL.STL
- link ZL: geometry collision mesh filename=file://PLACEHOLDER/ZL.STL; visual mesh filename=file://PLACEHOLDER/ZL.STL
- link base_link: geometry collision mesh filename=file://PLACEHOLDER/base_link.STL; visual mesh filename=file://PLACEHOLDER/base_link.STL
- link jaw0: geometry collision mesh filename=file://PLACEHOLDER/jaw0.STL; visual mesh filename=file://PLACEHOLDER/jaw0.STL
- link jaw1: geometry collision mesh filename=file://PLACEHOLDER/jaw1.STL; visual mesh filename=file://PLACEHOLDER/jaw1.STL

File: scara_ws/src/scara_description/scara (copy).urdf (robot description, URDF)
Before this commit: robot scara, 8 links, 7 joints
Links:
- link AL: geometry collision mesh filename=file:///home/ben/scara_ws/src/scara_description/AL.STL; visual mesh filename=file:///home/ben/scara_ws/src/scara_description/AL.STL
- link XL: geometry collision mesh filename=file:///home/ben/scara_ws/src/scara_description/XL.STL; visual mesh filename=file:///home/ben/scara_ws/src/scara_description/XL.STL
- link YL: geometry collision mesh filename=file:///home/ben/scara_ws/src/scara_description/YL.STL; visual mesh filename=file:///home/ben/scara_ws/src/scara_description/YL.STL
- link ZL: geometry collision mesh filename=file:///home/ben/scara_ws/src/scara_description/ZL.STL; visual mesh filename=file:///home/ben/scara_ws/src/scara_description/ZL.STL
- link base_link: geometry collision mesh filename=file:///home/ben/scara_ws/src/scara_description/base_link.S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; visual mesh filename=file:~/scara_description_symlink/base_link.STL
- link jaw0: geometry collision mesh filename=file:///home/ben/scara_ws/src/scara_description/jaw0.STL; visual mesh filename=file:///home/ben/scara_ws/src/scara_description/jaw0.STL
- link jaw1: geometry collision mesh filename=file:///home/ben/scara_ws/src/scara_description/jaw1.STL; visual mesh filename=file:///home/ben/scara_ws/src/scara_description/jaw1.STL
